Commit message: Lidar

File: models/iris/iris_base.xacro (robot description, xacro)
@@ -33,4 +33,6 @@
   <!-- Instantiate iris "mechanics" -->
   <xacro:include filename="$(arg rotors_description_dir)/iris/iris.xacro" />
+  <xacro:include filename="$(find velodyne_description)/urdf/HDL-32E.urdf.xacro"/>
+  <xacro:include filename="$(find velodyne_description)/urdf/VLP-16.urdf.xacro"/>
   <xacro:if value="$(arg enable_wind)">
     <xacro:wind_plugin_macro
@@ -122,4 +124,22 @@
   <origin xyz="0.02 0 0.07" rpy="0 0 0"/>
   </xacro:vi_sensor_depth_macro>
+  <!--xacro:HDL-32E
+    parent="base_link"
+    name="iris_$(arg drone_id)_velodyne"
+    topic="/iris_$(arg drone_id)/velodyne_points"
+    hz="10"
+    samples="220"
+  >
+  <origin xyz="-0.2 0 0.15" rpy="0 0 0" />
+  </xacro:HDL-32E-->
+  <VLP-16
+    name="${namespace}/VLP-16"
+    parent="base_link"
+    topic="/uav$(arg drone_id)/velodyne_points"
+    hz="10"
+    samples="220"
+  >
+  <origin xyz="0 0 0.07" rpy="0 0 0" />
+  </VLP-16>
   <!-- Mount an ADIS16448 IMU. -->
   <xacro:imu_plugin_macro
