Commit message: Added building and orb_slam2

File: models/component_snippets.xacro (robot description, xacro)
@@ -416,12 +416,19 @@
   <!-- Macro to add a depth camera on the VI-sensor. -->
   <xacro:macro name="vi_sensor_depth_macro"
-    params="namespace parent_link camera_suffix frame_rate *origin">
+    params="namespace parent_link camera_suffix frame_rate *cylinder *origin">
     <link name="${namespace}/camera_${camera_suffix}_link">
       <collision>
         <origin xyz="0 0 0" rpy="0 0 0" />
         <geometry>
-          <cylinder length="0.01" radius="0.007" />
+          <xacro:insert_block name="cylinder" />
         </geometry>
       </collision>
+        <visual>
+          <origin xyz="0 0 0" rpy="0 1.57079632679 0" />
+          <geometry>
+            <xacro:insert_block name="cylinder" />
+          </geometry>
+          <material name="red" />
+        </visual>
       <inertial>
         <mass value="1e-5" />
@@ -451,5 +458,5 @@
           <horizontal_fov>2</horizontal_fov>
           <image>
-            <format>L8</format>
+            <format>R8G8B8</format>
             <width>640</width>
             <height>480</height>

File: models/iris/iris_base.xacro (robot description, xacro)
@@ -122,17 +122,18 @@
     frame_rate="30.0"
   >
-  <origin xyz="0.02 0 0.07" rpy="0 0 0"/>
+  <box size="0.05 0.05 0.05" />
+  <origin xyz="0 0 0.12" rpy="0 0 0"/>
   </xacro:vi_sensor_depth_macro>
-  <!--xacro:HDL-32E
+  <xacro:HDL-32E
     parent="base_link"
-    name="iris_$(arg drone_id)_velodyne"
-    topic="/iris_$(arg drone_id)/velodyne_points"
+    name="${namespace}/lidar$(arg drone_id)_VLP-16"
+    topic="/uav$(arg drone_id)/velodyne_points"
     hz="10"
     samples="220"
   >
   <origin xyz="-0.2 0 0.15" rpy="0 0 0" />
-  </xacro:HDL-32E-->
-  <VLP-16
-    name="${namespace}/VLP-16"
+  </xacro:HDL-32E>
+  <!--VLP-16
+    name="${namespace}/lidar$(arg drone_id)_VLP-16"
     parent="base_link"
     topic="/uav$(arg drone_id)/velodyne_points"
@@ -141,5 +142,5 @@
   >
   <origin xyz="0 0 0.07" rpy="0 0 0" />
-  </VLP-16>
+  </VLP-16-->
   <!-- Mount an ADIS16448 IMU. -->
   <xacro:imu_plugin_macro

Commit message: New repo

File: models/component_snippets.xacro (robot description, xacro)
@@ -425,5 +425,5 @@
       </collision>
         <visual>
-          <origin xyz="0 0 0" rpy="0 1.57079632679 0" />
+          <origin xyz="0 0 0" rpy="0 0 0" />
           <geometry>
             <xacro:insert_block name="cylinder" />
